File: leiterplatte_kuechenlicht.brd (EAGLE design)
At the start: 100 x 80 mm, 20 parts, among them IC1 MEGA8-P, IC2 7805TV

Commit message: 1
Parts:
- added R3, R4, R5: 16,4k, rcl:0204/7
- added S2, S3, S4: (no value), switch-omron:B3F-10XX
- moved C3 178.6 mm to (36.8, 43.2)
- moved S1 178.3 mm to (48.3, 45.7), turned to 90 degrees
- moved C7 177.3 mm to (34.3, 38.1), turned to 180 degrees
- moved POT_BRI 176.0 mm to (61.0, 5.08)
- moved R1 174.8 mm to (50.8, 57.1), turned to 90 degrees
- moved R2 170.7 mm to (36.8, 48.3)
- moved C2 165.7 mm to (34.3, 17.8), turned to 180 degrees
- moved C1 161.2 mm to (30.5, 21.6), turned to 270 degrees
- moved PT4115_R 133.6 mm to (81.3, 71.1), turned to 270 degrees
- moved PT4115_B 127.6 mm to (96.5, 71.1), turned to 270 degrees
- moved POT_SAT 114.2 mm to (38.1, 5.08)
- moved POT_COL 113.0 mm to (15.2, 5.08)
- moved PT4115_G 109.0 mm to (66.0, 71.1), turned to 270 degrees
- moved SV1 103.4 mm to (67.3, 30.5), turned to 90 degrees
- moved C5 83.6 mm to (43.2, 72.4), turned to 90 degrees
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Connections:
- new net N$15: IC1.3, R4.2, S3.2
- new net N$17: IC1.4, R5.2, S4.1, S4.2
- new net N$19: IC1.2, R3.2, S2.1, S2.2
- net +5V: now also R3.1, R4.1, R5.1
- net GND: now also S2.3, S2.4, S3.3, S3.4, S4.3, S4.4, SV1.6
- net N$4: now also IC1.24; no longer IC1.23
- net N$5: now also IC1.23; no longer IC1.24
Routing:
- net GND: track 0.00 -> 286.5 mm
- net +5V: track 0.00 -> 281.0 mm
- net N$7: track 0.00 -> 115.6 mm
- net N$12: track 0.00 -> 113.1 mm
- net N$13: track 0.00 -> 110.6 mm
- net N$2: track 0.00 -> 90.3 mm
- net N$6: track 0.00 -> 39.4 mm
- net N$8: track 0.00 -> 36.3 mm
- net N$4: track 0.00 -> 24.1 mm, vias 0 -> 2
- net N$3: track 0.00 -> 8.89 mm
- net N$17: track 0.00 -> 8.61 mm
- net N$19: track 0.00 -> 7.19 mm
- net N$15: track 0.00 -> 7.19 mm
- net N$1: track 0.00 -> 6.07 mm
Other:
- board size 100 x 80 mm -> 125.4 x 80 mm

Commit message: 2
Parts:
- C3: device capacitor-wima:C2.5-3 -> rcl:C050-025X075
- POT_BRI, POT_COL, POT_SAT: value (none) -> 10k
- moved SV1 44.2 mm to (25.4, 44.5), turned to 0 degrees
- moved C3 2.84 mm to (38.1, 45.7)
- moved R2 2.54 mm to (39.4, 48.3)
Connections:
- removed net N$17: IC1.4, R5.2, S4.1, S4.2
- new net N$14: IC1.2, R5.2, S4.1, S4.2
- net N$19: now also IC1.4; no longer IC1.2
Routing:
- net GND: track 286.5 -> 382.6 mm
- net N$19: track 7.19 -> 93.7 mm
- net N$15: track 7.19 -> 72.0 mm
- net N$14: track 0.00 -> 63.9 mm
- net N$5: track 0.00 -> 44.4 mm
- net N$11: track 0.00 -> 30.3 mm
- net N$9: track 0.00 -> 17.6 mm
- net N$10: track 0.00 -> 17.6 mm
- net N$8: track 36.3 -> 46.4 mm
- net N$17: track 8.61 -> 0.00 mm
- net N$1: track 6.07 -> 3.53 mm
- net +5V: track 281.0 -> 282.2 mm, vias 0 -> 3
- net N$4: vias 2 -> 0
