File: leiterplatte_kuechenlicht.sch (EAGLE design)
At the start: 26 parts, among them IC1 MEGA8-P, IC2 7805TV

Commit message: 2
Parts:
- C3: device capacitor-wima:C2,5-3 -> rcl:C-EU050-025X075
- POT_BRI, POT_COL, POT_SAT: value (none) -> 10k
Connections:
- removed net N$17: IC1.PD2(INT0), R5.2, S4.S, S4.S1
- new net N$14: IC1.PD0(RXD), R5.2, S4.S, S4.S1
- net N$19: now also IC1.PD2(INT0); no longer IC1.PD0(RXD)
Changed lines of the file:
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@@
 <setting verticaltext="up"/>
 </settings>
-<grid distance="0.05" unitdist="inch" unit="inch" style="lines" multiple="1" display="yes" altdistance="0.025" altunitdist="inch" altunit="inch"/>
+<grid distance="0.1" unitdist="inch" unit="inch" style="lines" multiple="1" display="no" altdistance="0.01" altunitdist="inch" altunit="inch"/>
 <layers>
 <layer number="1" name="Top" color="4" fill="1" visible="no" active="no"/>
@@
 <part name="GND1" library="supply1" deviceset="GND" device=""/>
 <part name="GND2" library="supply1" deviceset="GND" device=""/>
-<part name="POT_SAT" library="pot" deviceset="TRIM_EU-" device="CIP20C-6MM"/>
-<part name="POT_COL" library="pot" deviceset="TRIM_EU-" device="CIP20C-6MM"/>
-<part name="POT_BRI" library="pot" deviceset="TRIM_EU-" device="CIP20C-6MM"/>
+<part name="POT_SAT" library="pot" deviceset="TRIM_EU-" device="CIP20C-6MM" value="10k"/>
+<part name="POT_COL" library="pot" deviceset="TRIM_EU-" device="CIP20C-6MM" value="10k"/>
+<part name="POT_BRI" library="pot" deviceset="TRIM_EU-" device="CIP20C-6MM" value="10k"/>
 <part name="SUPPLY4" library="supply2" deviceset="+5V" device=""/>
 <part name="GND4" library="supply1" deviceset="GND" device=""/>
@@
 <part name="GND6" library="supply1" deviceset="GND" device=""/>
 <part name="C2" library="capacitor-wima" deviceset="C" device="2,5-3" value="100nF"/>
-<part name="C3" library="capacitor-wima" deviceset="C" device="2,5-3" value="47nF"/>
+<part name="C3" library="rcl" deviceset="C-EU" device="050-025X075" value="47nF"/>
 <part name="C7" library="capacitor-wima" deviceset="C" device="2,5-3" value="100nF"/>
 <part name="GND7" library="supply1" deviceset="GND" device=""/>
@@
 <pinref part="R3" gate="G$1" pin="2"/>
 <wire x1="196.85" y1="97.79" x2="194.31" y2="97.79" width="0.1524" layer="91"/>
-<pinref part="IC1" gate="G$1" pin="PD0(RXD)"/>
-<wire x1="147.32" y1="81.28" x2="182.88" y2="81.28" width="0.1524" layer="91"/>
-<wire x1="182.88" y1="81.28" x2="182.88" y2="97.79" width="0.1524" layer="91"/>
+<wire x1="182.88" y1="76.2" x2="182.88" y2="97.79" width="0.1524" layer="91"/>
 <wire x1="182.88" y1="97.79" x2="194.31" y2="97.79" width="0.1524" layer="91"/>
 <junction x="194.31" y="97.79"/>
+<pinref part="IC1" gate="G$1" pin="PD2(INT0)"/>
+<wire x1="182.88" y1="76.2" x2="147.32" y2="76.2" width="0.1524" layer="91"/>
 </segment>
 </net>
@@
 </segment>
 </net>
-<net name="N$17" class="0">
+<net name="N$14" class="0">
 <segment>
 <pinref part="R5" gate="G$1" pin="2"/>
@@
 <wire x1="219.71" y1="87.63" x2="219.71" y2="85.09" width="0.1524" layer="91"/>
 <junction x="218.44" y="87.63"/>
-<pinref part="IC1" gate="G$1" pin="PD2(INT0)"/>
-<wire x1="147.32" y1="76.2" x2="199.39" y2="76.2" width="0.1524" layer="91"/>
-<wire x1="199.39" y1="76.2" x2="199.39" y2="66.04" width="0.1524" layer="91"/>
-<wire x1="199.39" y1="66.04" x2="224.79" y2="66.04" width="0.1524" layer="91"/>
+<wire x1="172.72" y1="66.04" x2="224.79" y2="66.04" width="0.1524" layer="91"/>
 <wire x1="224.79" y1="66.04" x2="224.79" y2="87.63" width="0.1524" layer="91"/>
 <wire x1="224.79" y1="87.63" x2="219.71" y2="87.63" width="0.1524" layer="91"/>
 <junction x="219.71" y="87.63"/>
+<wire x1="172.72" y1="66.04" x2="172.72" y2="81.28" width="0.1524" layer="91"/>
+<pinref part="IC1" gate="G$1" pin="PD0(RXD)"/>
+<wire x1="172.72" y1="81.28" x2="147.32" y2="81.28" width="0.1524" layer="91"/>
 </segment>
 </net>
@@
 </sheet>
 </sheets>
+<errors>
+</errors>
 </schematic>
 </drawing>
